File: front-end/pcb/gps.sch (KiCad schematic (older format))
At the start: 116 parts, among them J1 USB, K101 CONTACTPAD, K102 CONTACTPAD

Commit message: edited some footprints, tracing pcb
Parts:
- removed VD3, VD5, VD7: LED, symbol LED
Other:
- moved on the sheet: R57, VD2, VD4, VD6
