File: front-end/pcb/glonass_rx.sch (KiCad schematic (older format))
At the start: 113 parts, among them J1 USB, K101 CONTACTPAD, K102 CONTACTPAD

Commit message: edited pcb one more time for Rezonit(0.225mm clearence for polygons), updated gerbers, filled all values in schematic
Parts:
- C43: value CAPP -> 10u
- DD1: value IC_24_XX -> 24LC128-I/SN
- DD2: value IC_CY7C68013A -> CY7C68013A-56PVXC
- DD3: value IC_XC9572XL -> XC9572XL-10VQG64I
- G101: value GXO-U108L -> GXO-U108L 25.0MHz
- J1: value USB -> USBB-1J
- R55, R56, R57: value RES -> 100
- R60: value RES -> PLD-2
- VD2, VD4, VD6: value LED -> KP-1608SURC
- XP6: value JTAG -> BH2-14
- XT1: value CRYSTAL -> HC-49SM 24.0MHz
- Z101, Z102, Z103, Z104, Z105: value BLM18 -> BLM18EG601SN1
Changed lines of the file:
@@
 LIBS:lib_connectors
 LIBS:lib_passive
+LIBS:glonass_rx-cache
 EELAYER 27 0
 EELAYER END
@@
 Sheet 1 1
 Title ""
-Date "5 mar 2015"
+Date "11 mar 2015"
 Rev ""
 Comp ""
@@
 P 30750 14850
 F 0 "VD6" H 30850 14950 60  0000 C CNN
-F 1 "LED" H 31225 15000 60  0000 C CNN
+F 1 "KP-1608SURC" H 31225 15000 60  0000 C CNN
 F 2 "" H 30750 14850 60  0001 C CNN
 F 3 "" H 30750 14850 60  0001 C CNN
@@
 P 30750 14050
 F 0 "VD2" H 30850 14150 60  0000 C CNN
-F 1 "LED" H 31225 14200 60  0000 C CNN
+F 1 "KP-1608SURC" H 31225 14200 60  0000 C CNN
 F 2 "" H 30750 14050 60  0001 C CNN
 F 3 "" H 30750 14050 60  0001 C CNN
@@
 P 12350 16150
 F 0 "C43" H 12450 16050 60  0000 C CNN
-F 1 "CAPP" H 12500 15800 60  0000 C CNN
+F 1 "10u" H 12500 15800 60  0000 C CNN
 F 2 "" H 12350 16150 60  0001 C CNN
 F 3 "" H 12350 16150 60  0001 C CNN
@@
 P 31500 17500
 F 0 "R60" H 31750 17625 60  0000 C CNN
-F 1 "RES" H 32000 17625 60  0000 C CNN
+F 1 "PLD-2" H 32000 17625 60  0000 C CNN
 F 2 "" H 31500 17500 60  0001 C CNN
 F 3 "" H 31500 17500 60  0001 C CNN
@@
 P 29900 14850
 F 0 "R57" H 30150 14975 60  0000 C CNN
-F 1 "RES" H 30400 14975 60  0000 C CNN
+F 1 "100" H 30400 14975 60  0000 C CNN
 F 2 "" H 29900 14850 60  0001 C CNN
 F 3 "" H 29900 14850 60  0001 C CNN
@@
 P 29900 14450
 F 0 "R56" H 30150 14575 60  0000 C CNN
-F 1 "RES" H 30400 14575 60  0000 C CNN
+F 1 "100" H 30400 14575 60  0000 C CNN
 F 2 "" H 29900 14450 60  0001 C CNN
 F 3 "" H 29900 14450 60  0001 C CNN
@@
 P 29900 14050
 F 0 "R55" H 30150 14175 60  0000 C CNN
-F 1 "RES" H 30400 14175 60  0000 C CNN
+F 1 "100" H 30400 14175 60  0000 C CNN
 F 2 "" H 29900 14050 60  0001 C CNN
 F 3 "" H 29900 14050 60  0001 C CNN
@@
 P 24400 15900
 F 0 "XP6" H 24650 16000 60  0000 C CNN
-F 1 "JTAG" H 24800 15300 60  0000 C CNN
+F 1 "BH2-14" H 24800 15300 60  0000 C CNN
 F 2 "" H 24400 15900 60  0001 C CNN
 F 3 "" H 24400 15900 60  0001 C CNN
@@
 P 20150 4000
 F 0 "J1" H 20150 4400 50  0000 C CNN
-F 1 "USB" H 20150 4050 50  0000 C CNN
+F 1 "USBB-1J" H 20150 4050 50  0000 C CNN
 F 2 "" H 20150 4000 60  0001 C CNN
 F 3 "" H 20150 4000 60  0001 C CNN
@@
 P 20650 5250
 F 0 "XT1" H 20950 5450 60  0000 C CNN
-F 1 "CRYSTAL" H 20950 5050 60  0000 C CNN
+F 1 "HC-49SM 24.0MHz" H 20950 5050 60  0000 C CNN
 F 2 "" H 20650 5250 60  0001 C CNN
 F 3 "" H 20650 5250 60  0001 C CNN
@@
 P 17750 3300
 F 0 "DD1" H 18250 3450 60  0000 C CNN
-F 1 "IC_24_XX" H 18250 2850 60  0000 C CNN
+F 1 "24LC128-I/SN" H 18250 2850 60  0000 C CNN
 F 2 "" H 17750 3300 60  0001 C CNN
 F 3 "" H 17750 3300 60  0001 C CNN
@@
 P 19550 4900
 F 0 "DD2" H 20350 5050 60  0000 C CNN
-F 1 "IC_CY7C68013A" H 20350 1850 60  0000 C CNN
+F 1 "CY7C68013A-56PVXC" H 20350 1850 60  0000 C CNN
 F 2 "" H 19550 4900 60  0001 C CNN
 F 3 "" H 19550 4900 60  0001 C CNN
@@
 P 27550 14000
 F 0 "DD3" H 28200 14150 60  0000 C CNN
-F 1 "IC_XC9572XL" H 28200 10200 60  0000 C CNN
+F 1 "XC9572XL-10VQG64I" H 28200 10200 60  0000 C CNN
 F 2 "" H 27550 14000 60  0001 C CNN
 F 3 "" H 27550 14000 60  0001 C CNN
@@
 P 4450 4650
 F 0 "G101" H 5100 4800 60  0000 C CNN
-F 1 "GXO-U108L" H 5100 4400 60  0000 C CNN
+F 1 "GXO-U108L 25.0MHz" H 5100 4400 60  0000 C CNN
 F 2 "" H 4450 4650 60  0000 C CNN
 F 3 "" H 4450 4650 60  0000 C CNN
@@
 P 5650 12700
 F 0 "Z101" H 6050 12850 60  0000 C CNN
-F 1 "BLM18" H 6050 12600 60  0000 C CNN
+F 1 "BLM18EG601SN1" H 6050 12600 60  0000 C CNN
 F 2 "" H 5650 12700 60  0000 C CNN
 F 3 "" H 5650 12700 60  0000 C CNN
@@
 P 5750 14050
 F 0 "Z102" H 6150 14200 60  0000 C CNN
-F 1 "BLM18" H 6150 13950 60  0000 C CNN
+F 1 "BLM18EG601SN1" H 6150 13950 60  0000 C CNN
 F 2 "" H 5750 14050 60  0000 C CNN
 F 3 "" H 5750 14050 60  0000 C CNN
@@
 P 5750 15250
 F 0 "Z103" H 6150 15400 60  0000 C CNN
-F 1 "BLM18" H 6150 15150 60  0000 C CNN
+F 1 "BLM18EG601SN1" H 6150 15150 60  0000 C CNN
 F 2 "" H 5750 15250 60  0000 C CNN
 F 3 "" H 5750 15250 60  0000 C CNN
@@
 P 5750 16450
 F 0 "Z104" H 6150 16600 60  0000 C CNN
-F 1 "BLM18" H 6150 16350 60  0000 C CNN
+F 1 "BLM18EG601SN1" H 6150 16350 60  0000 C CNN
 F 2 "" H 5750 16450 60  0000 C CNN
 F 3 "" H 5750 16450 60  0000 C CNN
@@
 P 5750 17650
 F 0 "Z105" H 6150 17800 60  0000 C CNN
-F 1 "BLM18" H 6150 17550 60  0000 C CNN
+F 1 "BLM18EG601SN1" H 6150 17550 60  0000 C CNN
 F 2 "" H 5750 17650 60  0000 C CNN
 F 3 "" H 5750 17650 60  0000 C CNN
@@
 P 30750 14450
 F 0 "VD4" H 30850 14550 60  0000 C CNN
-F 1 "LED" H 31225 14600 60  0000 C CNN
+F 1 "KP-1608SURC" H 31225 14600 60  0000 C CNN
 F 2 "" H 30750 14450 60  0001 C CNN
 F 3 "" H 30750 14450 60  0001 C CNN
